Commit message: added mUseAVT option

File: sxr-avatar/app/src/main/assets/female/FemaleBody.urdf (robot description, URDF)
Before this commit: robot FemaleBody, 41 links, 40 joints
Links:
- link hair_02_01_JNT: geometry collision box size=0.030000 0.080000 0.150000
- link hair_02_02_JNT: geometry collision box size=0.080000 0.050000 0.150000
- link hair_02_JNT: geometry collision box size=0.050000 0.100000 0.170000
- link hair_03_01_JNT: geometry collision box size=0.150000 0.100000 0.030000
- link hair_03_02_JNT: geometry collision box size=0.150000 0.100000 0.050000
- link hair_03_JNT: geometry collision box size=0.150000 0.100000 0.030000
- link hair_04_01_JNT: geometry collision box size=0.030000 0.080000 0.150000
- link hair_04_02_JNT: geometry collision box size=0.080000 0.050000 0.150000
- link hair_04_JNT: geometry collision box size=0.050000 0.100000 0.170000
- link head_JNT: geometry collision cylinder length=0.321200 radius=0.186000
- link hips_JNT: geometry collision cylinder length=0.360000 radius=0.075000
- link l_arm_JNT: geometry collision cylinder length=0.390000 radius=0.040000
- link l_foot_JNT: geometry collision cylinder length=0.120000 radius=0.035000
- link l_forearm_JNT: geometry collision cylinder length=0.315000 radius=0.030000
- link l_hand_JNT: geometry collision cylinder length=0.270000 radius=0.035000
- link l_leg_JNT: geometry collision cylinder length=0.120000 radius=0.185000
- link l_shoulder_JNT: geometry collision cylinder length=0.195000 radius=0.060000
- link l_toebase_JNT: geometry collision cylinder length=0.060000 radius=0.035000
- link l_upleg_JNT: geometry collision cylinder length=0.165000 radius=0.160000
- link neck_JNT: geometry collision box size=0.061075 0.086617 0.040959
- link r_arm_JNT: geometry collision cylinder length=0.390000 radius=0.040000
- link r_foot_JNT: geometry collision cylinder length=0.120000 radius=0.035000
- link r_forearm_JNT: geometry collision cylinder length=0.315000 radius=0.030000
- link r_hand_JNT: geometry collision cylinder length=0.270000 radius=0.035000
- link r_leg_JNT: geometry collision cylinder length=0.120000 radius=0.185000
- link r_shoulder_JNT: geometry collision cylinder length=0.195000 radius=0.060000
- link r_toebase_JNT: geometry collision cylinder length=0.060000 radius=0.035000
- link r_upleg_JNT: geometry collision cylinder length=0.165000 radius=0.160000
- link spine2_JNT: geometry collision cylinder length=0.240000 radius=0.085000
- link spine_JNT: geometry collision cylinder length=0.210000 radius=0.160000

File: sxr-avatar/app/src/main/assets/hair/myemojihair_Long29_Male.urdf (robot description, URDF)
Before this commit: robot myemojihair_Long29_Male, 41 links, 39 joints
Links:
- removed link hips_JNT
- removed link l_arm_JNT
- removed link l_foot_JNT
- removed link l_forearm_JNT
- removed link l_hand_JNT
- removed link l_leg_JNT
- removed link l_shoulder_JNT
- removed link l_toebase_JNT
- removed link l_upleg_JNT
- removed link neck_JNT
- removed link r_arm_JNT
- removed link r_foot_JNT
- removed link r_forearm_JNT
- removed link r_hand_JNT
- removed link r_leg_JNT
- removed link r_shoulder_JNT
- removed link r_toebase_JNT
- removed link r_upleg_JNT
- removed link spine2_JNT
- removed link spine_JNT
- link hair_01_01_JNT: geometry collision box size=0.103646 0.059286 0.060867
- link hair_01_02_JNT: geometry collision box size=0.100000 0.066945 0.100000
- link hair_02_01_JNT: geometry collision box size=0.123627 0.071958 0.054122
- link hair_02_02_JNT: geometry collision box size=0.097416 0.050429 0.040728
- link hair_02_JNT: geometry collision box size=0.122910 0.065588 0.063352
- link hair_03_01_JNT: geometry collision box size=0.085890 0.070175 0.054122
- link hair_03_02_JNT: geometry collision box size=0.082071 0.051662 0.047039
- link hair_03_JNT: geometry collision box size=0.074002 0.065588 0.063352
- link hair_04_01_JNT: geometry collision box size=0.079377 0.068793 0.054122
- link hair_04_02_JNT: geometry collision box size=0.087849 0.042491 0.040728
- link hair_04_JNT: geometry collision box size=0.077194 0.065588 0.063352
- link hair_05_01_JNT: geometry collision box size=0.092047 0.070704 0.054122
- link hair_05_02_JNT: geometry collision box size=0.089752 0.043866 0.040728
- link hair_05_JNT: geometry collision box size=0.075838 0.065588 0.041787
- link hair_06_01_JNT: geometry collision box size=0.100000 0.072326 0.100000
- link hair_06_02_JNT: geometry collision box size=0.100000 0.062761 0.100000
- link head_JNT: geometry collision cylinder length=0.503874 radius=0.171667
Joints:
- removed joint joint_l_arm_JNT
- removed joint joint_l_foot_JNT
- removed joint joint_l_forearm_JNT
- removed joint joint_l_hand_JNT
- removed joint joint_l_leg_JNT
- removed joint joint_l_shoulder_JNT
- removed joint joint_l_toebase_JNT
- removed joint joint_l_upleg_JNT
- removed joint joint_neck_JNT
- removed joint joint_r_arm_JNT
- removed joint joint_r_foot_JNT
- removed joint joint_r_forearm_JNT
- removed joint joint_r_hand_JNT
- removed joint joint_r_leg_JNT
- removed joint joint_r_shoulder_JNT
- removed joint joint_r_toebase_JNT
- removed joint joint_r_upleg_JNT
- removed joint joint_spine2_JNT
- removed joint joint_spine_JNT
- joint joint_hair_01_01_JNT: origin xyz=0.000000 0.000000 0.000000 rpy=0.000000 0.000000 -0.000000 -> xyz=-0.007462 -0.040244 0.017889 rpy=36.283852 -5.260893 19.055040
- joint joint_hair_01_02_JNT: origin xyz=0.000000 0.000000 0.000000 rpy=0.000000 0.000000 -0.000000 -> xyz=0.007563 -0.015824 0.010678 rpy=-3.644172 3.087821 -2.064760
- joint joint_hair_01_JNT: origin xyz=0.000000 0.000000 0.000000 rpy=0.000000 0.000000 -0.000000 -> xyz=0.024220 0.018929 -0.004564 rpy=-34.457432 12.001139 -12.062184
- joint joint_hair_02_01_JNT: origin xyz=0.000000 0.000000 0.000000 rpy=0.000000 0.000000 -0.000000 -> xyz=-0.010744 -0.050459 0.015176 rpy=16.802267 10.918856 4.538116
- joint joint_hair_02_02_JNT: origin xyz=0.000000 0.000000 0.000000 rpy=0.000000 0.000000 -0.000000 -> xyz=-0.002559 -0.023522 0.003164 rpy=1.656937 5.027170 1.966421
- joint joint_hair_02_JNT: origin xyz=0.000000 0.000000 0.000000 rpy=0.000000 0.000000 -0.000000 -> xyz=0.028773 0.011384 -0.028946 rpy=-16.662157 -13.502582 -10.773018
- joint joint_hair_03_01_JNT: origin xyz=0.000000 0.000000 0.000000 rpy=0.000000 0.000000 -0.000000 -> xyz=0.011053 -0.092308 0.021056 rpy=1.003631 -14.664025 11.274240
- joint joint_hair_03_02_JNT: origin xyz=0.000000 0.000000 0.000000 rpy=0.000000 0.000000 -0.000000 -> xyz=0.001394 -0.036355 0.016730 rpy=2.522924 6.285172 1.045495
- joint joint_hair_03_JNT: origin xyz=0.000000 0.000000 0.000000 rpy=0.000000 0.000000 -0.000000 -> xyz=0.008288 0.027404 -0.047282 rpy=-1.198513 -13.988201 -5.719682
- joint joint_hair_04_01_JNT: origin xyz=0.000000 0.000000 0.000000 rpy=0.000000 0.000000 -0.000000 -> xyz=-0.002189 -0.079375 0.019609 rpy=-3.731254 -12.103778 -10.615581
- joint joint_hair_04_02_JNT: origin xyz=0.000000 0.000000 0.000000 rpy=0.000000 0.000000 -0.000000 -> xyz=0.005530 -0.041298 0.010227 rpy=1.181131 -9.287937 5.515448
- joint joint_hair_04_JNT: origin xyz=0.000000 0.000000 0.000000 rpy=0.000000 0.000000 -0.000000 -> xyz=-0.023260 0.007525 -0.089279 rpy=8.497117 -10.388098 7.432651
- joint joint_hair_05_01_JNT: origin xyz=0.000000 0.000000 0.000000 rpy=0.000000 0.000000 -0.000000 -> xyz=0.007170 -0.088832 -0.000131 rpy=-8.261026 14.359652 -1.293038
- joint joint_hair_05_02_JNT: origin xyz=0.000000 0.000000 0.000000 rpy=0.000000 0.000000 -0.000000 -> xyz=0.000326 -0.040389 -0.006885 rpy=-5.621805 15.238911 -1.515952
- joint joint_hair_05_JNT: origin xyz=0.000000 0.000000 0.000000 rpy=0.000000 0.000000 -0.000000 -> xyz=-0.053388 0.015039 -0.041469 rpy=22.122511 -26.466848 14.351749
- joint joint_hair_06_01_JNT: origin xyz=0.000000 0.000000 0.000000 rpy=0.000000 0.000000 -0.000000 -> xyz=0.031738 -0.011219 0.076471 rpy=-12.340368 -80.992996 -12.654504
- joint joint_hair_06_02_JNT: origin xyz=-0.066113 0.613543 0.103580 rpy=0.000000 0.000000 -0.000000 -> xyz=0.106174 -0.001378 0.275615 rpy=-8.752030 -6.779328 5.495333
- joint joint_hair_06_JNT: origin xyz=0.000000 0.000000 0.000000 rpy=0.000000 0.000000 -0.000000 -> xyz=-0.061150 0.025813 -0.003559 rpy=46.029663 17.864519 14.030622

Commit message: put hair back

File: sxr-avatar/app/src/main/assets/female/FemaleBody.urdf (robot description, URDF)
Before this commit: robot FemaleBody, 41 links, 40 joints
Links:
- link hair_02_01_JNT: geometry collision box size=0.030000 0.150000 0.080000
- link hair_02_02_JNT: geometry collision box size=0.080000 0.150000 0.050000
- link hair_02_JNT: geometry collision box size=0.050000 0.170000 0.100000
- link hair_03_01_JNT: geometry collision box size=0.150000 0.030000 0.100000
- link hair_03_02_JNT: geometry collision box size=0.150000 0.050000 0.100000
- link hair_03_JNT: geometry collision box size=0.150000 0.030000 0.100000
- link hair_04_01_JNT: geometry collision box size=0.030000 0.150000 0.080000
- link hair_04_02_JNT: geometry collision box size=0.080000 0.150000 0.050000
- link hair_04_JNT: geometry collision box size=0.050000 0.170000 0.100000
- link head_JNT: geometry collision capsule length=0.438000 radius=0.124000
- link hips_JNT: geometry collision capsule length=0.360000 radius=0.075000
- link l_arm_JNT: geometry collision capsule length=0.390000 radius=0.040000
- link l_foot_JNT: geometry collision capsule length=0.240000 radius=0.035000
- link l_forearm_JNT: geometry collision capsule length=0.315000 radius=0.030000
- link l_hand_JNT: geometry collision capsule length=0.270000 radius=0.035000
- link l_leg_JNT: geometry collision capsule length=0.555000 radius=0.035000
- link l_shoulder_JNT: geometry collision capsule length=0.195000 radius=0.060000
- link l_toebase_JNT: geometry collision capsule length=0.090000 radius=0.035000
- link l_upleg_JNT: geometry collision capsule length=0.480000 radius=0.055000
- link neck_JNT: geometry collision box size=0.061075 0.040959 0.086617
- link r_arm_JNT: geometry collision capsule length=0.390000 radius=0.040000
- link r_foot_JNT: geometry collision capsule length=0.240000 radius=0.035000
- link r_forearm_JNT: geometry collision capsule length=0.315000 radius=0.030000
- link r_hand_JNT: geometry collision capsule length=0.270000 radius=0.035000
- link r_leg_JNT: geometry collision capsule length=0.555000 radius=0.035000
- link r_shoulder_JNT: geometry collision capsule length=0.195000 radius=0.060000
- link r_toebase_JNT: geometry collision capsule length=0.090000 radius=0.035000
- link r_upleg_JNT: geometry collision capsule length=0.480000 radius=0.055000
- link spine2_JNT: geometry collision capsule length=0.255000 radius=0.093537
- link spine_JNT: geometry collision capsule length=0.480000 radius=0.090000
Joints:
- joint joint_hair_01_01_JNT: origin xyz=-0.000147 -0.047979 0.000491 rpy=0.000000 0.000000 -0.000000 -> xyz=-0.000147 -0.047979 0.000491 rpy=0.000000 0.000000 0.000000
- joint joint_hair_01_02_JNT: origin xyz=-0.000361 -0.117934 0.001208 rpy=0.000000 0.000000 -0.000000 -> xyz=-0.000361 -0.117934 0.001208 rpy=0.000000 0.000000 0.000000
- joint joint_hair_01_JNT: origin xyz=0.000870 0.101516 0.145076 rpy=0.000000 0.000000 -0.000000 -> xyz=0.000870 0.101516 0.145076 rpy=0.000000 0.000000 0.000000
- joint joint_hair_02_01_JNT: origin xyz=0.000294 -0.095958 0.000983 rpy=0.000000 0.000000 -0.000000 -> xyz=0.000294 -0.095958 0.000983 rpy=0.000000 0.000000 0.000000
- joint joint_hair_02_02_JNT: origin xyz=0.000361 -0.117934 0.001208 rpy=0.000000 0.000000 -0.000000 -> xyz=0.000361 -0.117934 0.001208 rpy=0.000000 0.000000 0.000000
- joint joint_hair_02_JNT: origin xyz=-0.121400 0.147671 -0.031654 rpy=0.000000 0.000000 -0.000000 -> xyz=-0.121400 0.147671 -0.031654 rpy=0.000000 0.000000 0.000000
- joint joint_hair_03_01_JNT: origin xyz=-0.000294 -0.095957 0.000983 rpy=0.000000 0.000000 -0.000000 -> xyz=-0.000294 -0.095957 0.000983 rpy=0.000000 0.000000 0.000000
- joint joint_hair_03_02_JNT: origin xyz=-0.000361 -0.117935 0.001208 rpy=0.000000 0.000000 -0.000000 -> xyz=-0.000361 -0.117935 0.001208 rpy=0.000000 0.000000 0.000000
- joint joint_hair_03_JNT: origin xyz=0.001016 0.147194 -0.154358 rpy=0.000000 0.000000 -0.000000 -> xyz=0.001016 0.147194 -0.154358 rpy=0.000000 0.000000 0.000000
- joint joint_hair_04_01_JNT: origin xyz=-0.000294 -0.095958 0.000983 rpy=0.000000 0.000000 -0.000000 -> xyz=-0.000294 -0.095958 0.000983 rpy=0.000000 0.000000 0.000000
- joint joint_hair_04_02_JNT: origin xyz=-0.000361 -0.117934 0.001208 rpy=0.000000 0.000000 -0.000000 -> xyz=-0.000361 -0.117934 0.001208 rpy=0.000000 0.000000 0.000000
- joint joint_hair_04_JNT: origin xyz=0.122806 0.147671 -0.031654 rpy=0.000000 0.000000 -0.000000 -> xyz=0.122806 0.147671 -0.031654 rpy=0.000000 0.000000 0.000000
- joint joint_hair_05_01_JNT: origin xyz=0.000013 0.085706 -0.000878 rpy=0.000000 0.000000 -0.000000 -> xyz=0.000013 0.085706 -0.000878 rpy=0.000000 0.000000 0.000000
- joint joint_hair_05_02_JNT: origin xyz=0.000013 0.085707 -0.000878 rpy=0.000000 0.000000 -0.000000 -> xyz=0.000013 0.085707 -0.000878 rpy=0.000000 0.000000 0.000000
- joint joint_hair_05_JNT: origin xyz=0.068959 0.221359 0.006956 rpy=0.000000 0.000000 -0.000000 -> xyz=0.068959 0.221359 0.006956 rpy=0.000000 0.000000 0.000000
- joint joint_hair_06_01_JNT: origin xyz=0.000013 0.085706 -0.000878 rpy=0.000000 0.000000 -0.000000 -> xyz=0.000013 0.085706 -0.000878 rpy=0.000000 0.000000 0.000000
- joint joint_hair_06_02_JNT: origin xyz=0.000013 0.085707 -0.000878 rpy=0.000000 0.000000 -0.000000 -> xyz=0.000013 0.085707 -0.000878 rpy=0.000000 0.000000 0.000000
- joint joint_hair_06_JNT: origin xyz=-0.070810 0.221380 0.006956 rpy=0.000000 0.000000 -0.000000 -> xyz=-0.070810 0.221380 0.006956 rpy=0.000000 0.000000 0.000000
- joint joint_head_JNT: origin xyz=-0.000819 0.151035 0.021716 rpy=0.000000 0.000000 -0.000000 -> xyz=-0.000819 0.151035 0.021716 rpy=0.000000 0.000000 0.000000
- joint joint_l_arm_JNT: origin xyz=0.190469 0.002851 -0.001221 rpy=0.000000 0.000000 -0.000000 -> xyz=0.190469 0.002851 -0.001221 rpy=0.000000 0.000000 0.000000
- joint joint_l_earring_accessory_JNT: origin xyz=0.117393 -0.034802 -0.002251 rpy=0.000000 0.000000 -0.000000 -> xyz=0.117393 -0.034802 -0.002251 rpy=0.000000 0.000000 0.000000
- joint joint_l_foot_JNT: origin xyz=0.001447 -0.216052 0.046643 rpy=0.000000 0.000000 -0.000000 -> xyz=0.001447 -0.216052 0.046643 rpy=0.000000 0.000000 0.000000
- joint joint_l_forearm_JNT: axis 0.000000 1.000000 0.000000 -> 0.000000 0.000000 1.000000; origin xyz=0.240328 -0.000001 0.018851 rpy=0.000000 0.000000 -0.000000 -> xyz=0.240328 -0.000001 0.018851 rpy=0.000000 0.000000 0.000000
- joint joint_l_hand_JNT: origin xyz=0.145913 -0.006082 0.025126 rpy=0.000000 0.000000 -0.000000 -> xyz=0.145913 -0.006082 0.025126 rpy=0.000000 0.000000 0.000000
- joint joint_l_leg_JNT: origin xyz=0.002832 -0.384417 -0.010570 rpy=0.000000 0.000000 -0.000000 -> xyz=0.002832 -0.384417 -0.010570 rpy=0.000000 0.000000 0.000000
- joint joint_l_shoulder_JNT: origin xyz=0.085153 0.058688 -0.018444 rpy=0.000000 0.000000 -0.000000 -> xyz=0.085153 0.058688 -0.018444 rpy=0.000000 0.000000 0.000000
- joint joint_l_toebase_JNT: origin xyz=0.000098 -0.032490 0.059404 rpy=0.000000 0.000000 -0.000000 -> xyz=0.000098 -0.032490 0.059404 rpy=0.000000 0.000000 0.000000
- joint joint_l_upleg_JNT: origin xyz=0.081457 -0.208145 0.002232 rpy=0.000000 0.000000 -0.000000 -> xyz=0.081457 -0.208145 0.002232 rpy=0.000000 0.000000 0.000000
- joint joint_neck_JNT: origin xyz=-0.000132 0.148075 -0.002603 rpy=0.000000 0.000000 -0.000000 -> xyz=-0.000132 0.148075 -0.002603 rpy=0.000000 0.000000 0.000000
- joint joint_r_arm_JNT: origin xyz=-0.190469 0.002851 -0.001221 rpy=0.000000 0.000000 -0.000000 -> xyz=-0.190469 0.002851 -0.001221 rpy=0.000000 0.000000 0.000000
- joint joint_r_earring_accessory_JNT: origin xyz=-0.115987 -0.034802 -0.002251 rpy=0.000000 0.000000 -0.000000 -> xyz=-0.115987 -0.034802 -0.002251 rpy=0.000000 0.000000 0.000000
- joint joint_r_foot_JNT: origin xyz=-0.001447 -0.216052 0.046643 rpy=0.000000 0.000000 -0.000000 -> xyz=-0.001447 -0.216052 0.046643 rpy=0.000000 0.000000 0.000000
- joint joint_r_forearm_JNT: axis 0.000000 -1.000000 0.000000 -> 0.000000 0.000000 -1.000000; origin xyz=-0.240328 -0.000001 0.018851 rpy=0.000000 0.000000 -0.000000 -> xyz=-0.240328 -0.000001 0.018851 rpy=0.000000 0.000000 0.000000
- joint joint_r_hand_JNT: origin xyz=-0.145405 -0.005891 0.025118 rpy=0.000000 0.000000 -0.000000 -> xyz=-0.145405 -0.005891 0.025118 rpy=0.000000 0.000000 0.000000
- joint joint_r_leg_JNT: origin xyz=-0.002832 -0.384417 -0.010570 rpy=0.000000 0.000000 -0.000000 -> xyz=-0.002832 -0.384417 -0.010570 rpy=0.000000 0.000000 0.000000
- joint joint_r_shoulder_JNT: origin xyz=-0.085648 0.058688 -0.018444 rpy=0.000000 0.000000 -0.000000 -> xyz=-0.085648 0.058688 -0.018444 rpy=0.000000 0.000000 0.000000
- joint joint_r_toebase_JNT: origin xyz=-0.000098 -0.032490 0.059404 rpy=0.000000 0.000000 -0.000000 -> xyz=-0.000098 -0.032490 0.059404 rpy=0.000000 0.000000 0.000000
- joint joint_r_upleg_JNT: origin xyz=-0.081457 -0.208145 0.002232 rpy=0.000000 0.000000 -0.000000 -> xyz=-0.081457 -0.208145 0.002232 rpy=0.000000 0.000000 0.000000
- joint joint_spine2_JNT: origin xyz=0.000124 0.295181 -0.022932 rpy=0.000000 0.000000 -0.000000 -> xyz=0.000124 0.295181 -0.022932 rpy=0.000000 0.000000 0.000000
- joint joint_spine_JNT: origin xyz=0.000123 0.036636 -0.000207 rpy=0.000000 0.000000 -0.000000 -> xyz=0.000123 0.036636 -0.000207 rpy=0.000000 0.000000 0.000000
